File: Doppler_Debug_Brd/Radar/Radar.kicad_pcb (KiCad board)
At the start: 2 copper layers, 65 x 65 mm, 82 parts, among them J1 AVR-PDI-6, J2 USB_B, J3 338728-8, U1 LM3671MF-3.3/NOPB, U2 ATxmega256A3U-A, U3 FT231XS, U4 MCP6002-xMS, U5 MCP6004, U6 MCP6002-xMS, U7 MCP6004

Commit message: AB BRDlayout update
pinout radar module needs checking
Parts:
- added C33: DNM, Capacitor_SMD:C_0805_2012Metric_Pad1.18x1.45mm_HandSolder, F.Cu at (120.8, 86.5)
- added C34: DNM, Capacitor_SMD:C_0805_2012Metric_Pad1.18x1.45mm_HandSolder, F.Cu at (132.9, 95.2)
- added D10: RB751S40T1G, Diode_SMD:D_SOD-523, F.Cu at (113.4, 81.2)
- added D7: RB751S40T1G, Diode_SMD:D_SOD-523, F.Cu at (122.9, 78.3)
- added D8: RB751S40T1G, Diode_SMD:D_SOD-523, F.Cu at (122.8, 81.8)
- added D9: RB751S40T1G, Diode_SMD:D_SOD-523, F.Cu at (113.4, 78.5)
- added R30: DNM, Resistor_SMD:R_0805_2012Metric_Pad1.20x1.40mm_HandSolder, F.Cu at (114.5, 86.7)
- added R31: DNM, Resistor_SMD:R_0805_2012Metric_Pad1.20x1.40mm_HandSolder, F.Cu at (129.1, 95.2)
- added R32: 0R, Resistor_SMD:R_0805_2012Metric_Pad1.20x1.40mm_HandSolder, F.Cu at (114.5, 88.8)
- added R33: 0R, Resistor_SMD:R_0805_2012Metric_Pad1.20x1.40mm_HandSolder, F.Cu at (129.1, 93.2)
- added R34: 1M, Resistor_SMD:R_0805_2012Metric_Pad1.20x1.40mm_HandSolder, F.Cu at (131.4, 109.2)
- added R35: 1M, Resistor_SMD:R_0805_2012Metric_Pad1.20x1.40mm_HandSolder, F.Cu at (150.6, 75.8)
- added R36: 300k, Resistor_SMD:R_0805_2012Metric_Pad1.20x1.40mm_HandSolder, F.Cu at (160.4, 77.5)
- added R37: 300k, Resistor_SMD:R_0805_2012Metric_Pad1.20x1.40mm_HandSolder, F.Cu at (138.8, 109.3)
- added R38: 300k, Resistor_SMD:R_0805_2012Metric_Pad1.20x1.40mm_HandSolder, F.Cu at (160.6, 79.5)
- added R39: 300k, Resistor_SMD:R_0805_2012Metric_Pad1.20x1.40mm_HandSolder, F.Cu at (138.8, 111.4)
- added TP2: IF_I, TestPoint:TestPoint_Pad_D1.0mm, F.Cu at (129.8, 73.2)
- added TP3: IF_Q, TestPoint:TestPoint_Pad_D1.0mm, F.Cu at (134.2, 62.8)
- added TP4: ADC_Q, TestPoint:TestPoint_Pad_D1.0mm, F.Cu at (149.4, 72.0)
- added TP5: ADC_I, TestPoint:TestPoint_Pad_D1.0mm, F.Cu at (134.1, 90.2)
- added TP6: 3v3_I, TestPoint:TestPoint_Pad_D1.0mm, F.Cu at (113.8, 107.8)
- added TP7: 3v3_Q, TestPoint:TestPoint_Pad_D1.0mm, F.Cu at (140.3, 93.0)
- C11, C14: value 200pF -> 33pF
- C12, C15: value 2nF -> 1nF
- C17, C19: value 110pF -> 100pF
- C18, C20: value 1.1nF -> 1nF
- C22, C23: value 43pF -> 100pF
- C26, C29: value 10pF -> 100pF
- C27, C28: value 220uF -> 10uF; footprint Capacitor_SMD:CP_Elec_10x10 -> Capacitor_SMD:C_0805_2012Metric_Pad1.18x1.45mm_HandSolder
- C30, C31: value 2.7nF -> 1nF
- R10, R9: value 1M6 -> 430k
- R11, R12: value 150k -> 82k
- R13, R14: value 750k -> 820k
- R15, R16: value 390k -> 51k
- R17: value 390k -> 1M
- R18: value 390k -> 300k
- R19, R20: value 430k -> 43k
- R21: value 430k -> 300k
- R22: value 430k -> 1M
- R7, R8: value 56k -> 430k
- moved C28 20.9 mm to (125.6, 71.2), turned to 90 degrees
- moved C27 8.82 mm to (123.3, 71.2), turned to 90 degrees
- moved R16 1.95 mm to (131.5, 111.3)
- moved C26 0.88 mm to (160.4, 81.6)
- moved C3 0.36 mm to (164.6, 78.4)
- moved C13 0.27 mm to (118.4, 88.8)
- moved R18 0.22 mm to (131.7, 106.1)
- moved C1 0.21 mm to (165.3, 88.5)
Connections:
- R17 pad 2: Net-(C22-Pad1) -> Net-(R17-Pad2)
- R18 pad 1: Net-(C25-Pad1) -> Net-(R18-Pad1)
- R21 pad 1: Net-(C30-Pad1) -> Net-(R17-Pad2)
- R21 pad 2: Net-(C26-Pad1) -> Net-(C22-Pad1)
- R22 pad 2: Net-(C29-Pad1) -> Net-(R22-Pad2)
- R23 pad 2: Net-(C27-Pad2) -> Net-(C28-Pad1)
- R24 pad 1: Net-(C27-Pad2) -> Net-(C28-Pad1)
- R25 pad 2: Net-(C28-Pad2) -> Net-(C27-Pad1)
- R26 pad 1: Net-(C28-Pad2) -> Net-(C27-Pad1)
- U4 pad 1: Net-(C27-Pad1) -> Net-(C28-Pad2)
- U4 pad 2: Net-(C27-Pad1) -> Net-(C28-Pad2)
- U4 pad 6: Net-(C28-Pad1) -> Net-(C27-Pad2)
- U4 pad 7: Net-(C28-Pad1) -> Net-(C27-Pad2)
- U6 pad 2: Net-(R27-Pad1) -> Net-(R30-Pad1)
- U6 pad 3: Net-(C27-Pad2) -> Net-(C28-Pad1)
- U6 pad 5: Net-(C28-Pad2) -> Net-(C27-Pad1)
- U6 pad 6: Net-(R28-Pad2) -> Net-(R31-Pad1)
Routing:
- net Net-(C27-Pad1): track 6.78 -> 41.9 mm, vias 0 -> 4
- net Net-(C28-Pad2): track 31.2 -> 4.05 mm, vias 3 -> 0
- net Net-(R22-Pad2): track 0.00 -> 14.6 mm, vias 0 -> 2
- net Net-(C27-Pad2): track 28.5 -> 14.1 mm
- net Net-(C29-Pad1): track 12.3 -> 25.8 mm, vias 0 -> 2
- net Net-(R17-Pad2): track 0.00 -> 10.3 mm, vias 0 -> 2
- net Net-(R31-Pad1): track 0.00 -> 10.1 mm
- net Net-(C22-Pad1): track 9.00 -> 18.7 mm
- net Net-(R35-Pad2): track 0.00 -> 8.54 mm
- net Net-(R30-Pad1): track 0.00 -> 8.26 mm
- net ADC_Q: track 30.8 -> 38.8 mm, vias 2 -> 3
- net 3v3_I: track 2.24 -> 8.71 mm
- net ADC_I: track 25.7 -> 32.2 mm, vias 3 -> 4
- net Net-(C30-Pad1): track 4.55 -> 10.1 mm, vias 0 -> 2
- net Net-(C28-Pad1): track 38.7 -> 33.7 mm, vias 2 -> 4
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Other:
- board text added: "Doppler Debug Board Rev: AB"
- board text removed: "Doppler Debug Board Rev: AA"
