File: Doppler_Debug_Brd/Radar/Radar.kicad_sch (KiCad schematic)
At the start: 0 parts

Commit message: Finalized code
Other:
- title: Doppler Radar Controll Board -> Doppler Debug Board
Changed lines of the file:
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@@
   (paper "A4")
   (title_block
-    (title "Doppler Radar Controll Board")
-    (date "2023-01-25")
-    (rev "AA")
+    (title "Doppler Debug Board")
+    (date "2023-09-18")
+    (rev "AB")
     (company "CleanMobility")
   )
